Commit message: first commit

File: urdf/tnbd.urdf (robot description, URDF)
Before this commit: robot tnbd, 9 links, 8 joints
Links:
- added link base_footprint
Joints:
- added joint base_joint: type fixed, parent base_footprint, child base_link, origin xyz=0.0118828123771107 -0.0151599566389232 0.0203146741285486 rpy=0 0 0
- joint back_joint: limit lower=0 upper=0 effort=0 velocity=0 -> lower=-1.570796 upper=0 effort=0 velocity=0
- joint feed_joint: limit lower=0 upper=0 effort=0 velocity=0 -> lower=-0.802851 upper=0 effort=0 velocity=0
- joint front_joint: limit lower=0 upper=0 effort=0 velocity=0 -> lower=0 upper=2.000321 effort=0 velocity=0
